File: pcb/keypad.kicad_sch (KiCad schematic)
At the start: 4 parts, among them U1 74AHCT1G125, U2 XIAO-ESP32-C6-DIP

Commit message: Swap U1 level shifter to SN74AHCT1G125DBVR (SOT-23-5)
The SOT-353 part was hard to hand solder. Same 74AHCT1G125 pinout, so only
the footprint changes. U1 shifts 0.1 mm right and its traces are rerouted;
gerbers regenerated.
Parts:
- U1: footprint Package_TO_SOT_SMD:SOT-353_SC-70-5 -> Package_TO_SOT_SMD:SOT-23-5
Changed lines of the file:
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@@
 			)
 		)
-		(property "Footprint" "Package_TO_SOT_SMD:SOT-353_SC-70-5"
+		(property "Footprint" "Package_TO_SOT_SMD:SOT-23-5"
 			(at 66.04 59.69 0)
 			(hide yes)

Commit message: Use hand-soldering SOT-23-5 footprint for U1
Longer pads (1.56 x 0.65 mm) for easier hand soldering. Same position, pinout and routing; DRC unchanged.
Parts:
- U1: footprint Package_TO_SOT_SMD:SOT-23-5 -> Package_TO_SOT_SMD:SOT-23-5_HandSoldering
Changed lines of the file:
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@@
 			)
 		)
-		(property "Footprint" "Package_TO_SOT_SMD:SOT-23-5"
+		(property "Footprint" "Package_TO_SOT_SMD:SOT-23-5_HandSoldering"
 			(at 66.04 59.69 0)
 			(hide yes)
